Commit message: added new frame transform from ground_link and base_link

File: CER02/cer.urdf (robot description, URDF)
Before this commit: robot SIM_CER_ROBOT, 60 links, 59 joints
Links:
- added link ground_link
Joints:
- added joint ground_link_fixed_joint: type fixed, parent base_link, child ground_link, origin xyz=0 0 -0.2 rpy=0 0 0
