Commit message: Restored missing "ground_link" to cer.urdf files

File: R1SN000/cer.urdf (robot description, URDF)
Before this commit: robot SIM_CER_ROBOT, 58 links, 57 joints
Links:
- added link ground_link
Joints:
- added joint ground_link_fixed_joint: type fixed, parent base_link, child ground_link, origin xyz=0 0 -0.2 rpy=0 0 0

File: R1SN002/cer.urdf (robot description, URDF)
Before this commit: robot SIM_CER_ROBOT, 60 links, 59 joints
Links:
- added link ground_link
Joints:
- added joint ground_link_fixed_joint: type fixed, parent base_link, child ground_link, origin xyz=0 0 -0.2 rpy=0 0 0
